Commit message: Added a basic world

File: drone_sim/urdf/drone.urdf (robot description, URDF)
Before this commit: robot my_robot, 1 links, 0 joints
Links:
- link base_link: mass None -> 1.0; geometry collision mesh filename=package://drone_sim/meshes/drone.stl scale=0.001 0.001 0.001; visual mesh filename=package://drone_sim/meshes/drone.stl scale=0.001 0.001 0.001

Commit message: Changed the mass value

File: drone_sim/urdf/drone.urdf (robot description, URDF)
Before this commit: robot robot, 1 links, 0 joints
Links:
- link base_link: mass 1.0 -> 10.0

Commit message: Plugin works fine

File: drone_sim/urdf/drone.urdf (robot description, URDF)
Before this commit: robot my_robot, 1 links, 0 joints
Links:
- added link prop, mass 0.01; collision sphere radius=0.1; visual sphere radius=0.1
- added link prop2, mass 0.01; collision sphere radius=0.1; visual sphere radius=0.1
- added link prop3, mass 0.01; collision sphere radius=0.1; visual sphere radius=0.1
- added link prop4, mass 0.01; collision sphere radius=0.1; visual sphere radius=0.1
Joints:
- added joint prop1_joint: type revolute, parent base_link, child prop, origin xyz=0.105 0.105 0.0 rpy=0 0 0, axis 0 0 1, limit effort=1.0 velocity=100
- added joint prop2_joint: type revolute, parent base_link, child prop2, origin xyz=0.105 -0.105 0.0 rpy=0 0 0, axis 0 0 1, limit effort=1.0 velocity=100
- added joint prop3_joint: type revolute, parent base_link, child prop3, origin xyz=-0.105 -0.105 0.0 rpy=0 0 0, axis 0 0 1, limit effort=1.0 velocity=100
- added joint prop4_joint: type revolute, parent base_link, child prop4, origin xyz=-0.105 0.105 0.0 rpy=0 0 0, axis 0 0 1, limit effort=1.0 velocity=100

Commit message: Now the plugin works perfectly

File: drone_sim/urdf/drone.urdf (robot description, URDF)
Before this commit: robot my_robot, 5 links, 4 joints
Links:
- removed link prop
- added link prop1, mass 0.01; collision sphere radius=0.1; visual sphere radius=0.1
Joints:
- joint prop1_joint: child prop -> prop1; origin xyz=0.105 0.105 0.0 rpy=0 0 0 -> xyz=1.05 1.05 0.0 rpy=0 0 0
- joint prop2_joint: origin xyz=0.105 -0.105 0.0 rpy=0 0 0 -> xyz=1.05 -1.05 0.0 rpy=0 0 0
- joint prop3_joint: origin xyz=-0.105 -0.105 0.0 rpy=0 0 0 -> xyz=-1.05 -1.05 0.0 rpy=0 0 0
- joint prop4_joint: origin xyz=-0.105 0.105 0.0 rpy=0 0 0 -> xyz=-1.05 1.05 0.0 rpy=0 0 0

Commit message: Added code for testing mpc

File: drone_sim/urdf/drone.urdf (robot description, URDF)
Before this commit: robot my_robot, 5 links, 4 joints
Links:
- link base_link: geometry collision mesh filename=package://drone_sim/meshes/drone.dae scale=0.001 0.001 0.001; visual mesh filename=package://drone_sim/meshes/drone.dae scale=0.001 0.001 0.001
- link prop1: geometry collision sphere radius=0.001; visual sphere radius=0.001
- link prop2: geometry collision sphere radius=0.001; visual sphere radius=0.001
- link prop3: geometry collision sphere radius=0.001; visual sphere radius=0.001
- link prop4: geometry collision sphere radius=0.001; visual sphere radius=0.001
Joints:
- joint prop1_joint: origin xyz=1.05 1.05 0.0 rpy=0 0 0 -> xyz=0.105 0.105 0.0 rpy=0 0 0
- joint prop2_joint: origin xyz=1.05 -1.05 0.0 rpy=0 0 0 -> xyz=0.105 -0.105 0.0 rpy=0 0 0
- joint prop3_joint: origin xyz=-1.05 -1.05 0.0 rpy=0 0 0 -> xyz=-0.105 -0.105 0.0 rpy=0 0 0
- joint prop4_joint: origin xyz=-1.05 1.05 0.0 rpy=0 0 0 -> xyz=-0.105 0.105 0.0 rpy=0 0 0

Commit message: Basic test case is close to complete

File: drone_sim/urdf/drone.urdf (robot description, URDF)
Before this commit: robot my_robot, 5 links, 4 joints
Links:
- link base_link: mass 1.0 -> 1.2
- link prop1: mass 0.01 -> 0.0001
- link prop2: mass 0.01 -> 0.0001
- link prop3: mass 0.01 -> 0.0001
- link prop4: mass 0.01 -> 0.0001

Commit message: Forward dynamics works good, adding inverse dynamics

File: drone_sim/urdf/drone.urdf (robot description, URDF)
Before this commit: robot my_robot, 5 links, 4 joints
Joints:
- joint prop1_joint: origin xyz=0.105 0.105 0.0 rpy=0 0 0 -> xyz=0 -0.1484 0.0 rpy=0 0 0
- joint prop2_joint: origin xyz=0.105 -0.105 0.0 rpy=0 0 0 -> xyz=0.1484 0 0.0 rpy=0 0 0
- joint prop3_joint: origin xyz=-0.105 -0.105 0.0 rpy=0 0 0 -> xyz=-0 0.1484 0.0 rpy=0 0 0
- joint prop4_joint: origin xyz=-0.105 0.105 0.0 rpy=0 0 0 -> xyz=-0.1484 0. 0.0 rpy=0 0 0

Commit message: Added basic MPC

File: drone_sim/urdf/drone.urdf (robot description, URDF)
Before this commit: robot my_robot, 5 links, 4 joints
Joints:
- joint prop1_joint: origin xyz=0 -0.1484 0.0 rpy=0 0 0 -> xyz=0 -0.13181 0.0 rpy=0 0 0
- joint prop2_joint: origin xyz=0.1484 0 0.0 rpy=0 0 0 -> xyz=0.13181 0 0.0 rpy=0 0 0
- joint prop3_joint: origin xyz=-0 0.1484 0.0 rpy=0 0 0 -> xyz=-0 0.13181 0.0 rpy=0 0 0
- joint prop4_joint: origin xyz=-0.1484 0. 0.0 rpy=0 0 0 -> xyz=-0.13181 0. 0.0 rpy=0 0 0

Commit message: Implemented the plugin

File: drone_sim/urdf/drone.urdf (robot description, URDF)
Before this commit: robot my_robot, 5 links, 4 joints
Links:
- removed link prop1
- removed link prop2
- removed link prop3
- removed link prop4
- link base_link: geometry collision mesh filename=package://drone_sim/meshes/drone.stl scale=0.001 0.001 0.001; visual mesh filename=package://drone_sim/meshes/drone.stl scale=0.001 0.001 0.001
Joints:
- removed joint prop1_joint
- removed joint prop2_joint
- removed joint prop3_joint
- removed joint prop4_joint
